Commit message: Corregir 4 bloqueantes simulación: cámara URDF, paredes 7x7, TF cámara, use_sim_time EKF

File: src/osr-rover-code/ROS/osr_gazebo/urdf/gazebo.urdf.xacro (robot description, xacro)
@@ -167,4 +167,35 @@
     </plugin>
   </gazebo>
+  <!-- Cámara frontal para detección ArUco (Gazebo Harmonic) -->
+  <gazebo reference="camera">
+    <sensor name="camera_sensor" type="camera">
+      <always_on>true</always_on>
+      <update_rate>10</update_rate>
+      <visualize>true</visualize>
+      <topic>camera</topic>
+      <gz_frame_id>camera</gz_frame_id>
+      <camera>
+        <horizontal_fov>1.3962634</horizontal_fov>
+        <image>
+          <width>640</width>
+          <height>480</height>
+          <format>R8G8B8</format>
+        </image>
+        <clip>
+          <near>0.05</near>
+          <far>10.0</far>
+        </clip>
+        <noise>
+          <type>gaussian</type>
+          <mean>0.0</mean>
+          <stddev>0.005</stddev>
+        </noise>
+      </camera>
+    </sensor>
+  </gazebo>
+  <gazebo>
+    <plugin filename="gz-sim-sensors-system" name="gz::sim::systems::Sensors">
+    </plugin>
+  </gazebo>
   <gazebo>
     <plugin filename="gz-sim-odometry-publisher-system" name="gz::sim::systems::OdometryPublisher">

File: src/osr-rover-code/ROS/osr_gazebo/urdf/osr.urdf.xacro (robot description, xacro)
@@ -45,4 +45,16 @@
         <axis xyz="0 0 1"/>
     </joint>
+    <!-- Cámara frontal para detección ArUco -->
+    <link name="camera">
+        <inertial>
+            <mass value="0.01"/>
+            <inertia ixx="0.0" ixy="0.0" ixz="0.0" iyy="0.0" iyz="0.0" izz="0.0"/>
+        </inertial>
+    </link>
+    <joint name="camera_joint" type="fixed">
+        <parent link="base_link"/>
+        <child link="camera"/>
+        <origin rpy="0 0 0" xyz="0.09 0.0 0.2"/>
+    </joint>
     <link name="box_rotate">
         <collision>
